File: Hardware/phase.kicad_sch (KiCad schematic)
At the start: 12 parts, among them Q1 AP30H80Q, Q2 AP30H80Q, U2 INA181A1IDBVR

Commit message: Reannotated
Parts:
- renumbered C13 to C25, C12 to C27, C14 to C4, D6 to D11, Q1 to Q16, Q2 to Q18, R6 to R2, R3 to R30, R4 to R32, R12 to R4, R13 to R6

Commit message: Pretty much all components now have values
Parts:
- C25: value C -> 10u
- C27, C4: value C -> 100n
- D11: value D_Schottky -> B5819WS
- R2: value R -> 0R01
- R30, R32: value R -> 2R2
- R4, R6: value R -> 1k
Changed lines of the file:
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@@
 			)
 		)
-		(property "Value" "R"
+		(property "Value" "1k"
 			(at 146.558 88.8421 0)
 			(effects
@@
 			)
 		)
-		(property "Value" "C"
+		(property "Value" "10u"
 			(at 101.3841 78.6757 0)
 			(effects
@@
 			)
 		)
-		(property "Value" "C"
+		(property "Value" "100n"
 			(at 72.1741 87.5657 0)
 			(effects
@@
 			)
 		)
-		(property "Value" "R"
+		(property "Value" "2R2"
 			(at 78.74 85.09 90)
 			(effects
@@
 			)
 		)
-		(property "Value" "R"
+		(property "Value" "0R01"
 			(at 116.84 89.9738 90)
 			(effects
@@
 			)
 		)
-		(property "Value" "D_Schottky"
+		(property "Value" "B5819WS"
 			(at 71.882 67.5696 90)
 			(effects
@@
 			)
 		)
-		(property "Value" "R"
+		(property "Value" "2R2"
 			(at 78.74 110.49 90)
 			(effects
@@
 			)
 		)
-		(property "Value" "C"
+		(property "Value" "100n"
 			(at 142.0241 64.7057 0)
 			(effects
@@
 			)
 		)
-		(property "Value" "R"
+		(property "Value" "1k"
 			(at 146.558 101.5421 0)
 			(effects

Commit message: Second cut of circuit board
Parts:
- C27, C4: footprint (none) -> Capacitor_SMD:C_0603_1608Metric
- D11: footprint (none) -> Diode_SMD:D_SOD-323
- Q16, Q18: footprint :DFN-8_L3.2-W3.1-P0.65-LS3.4-BL -> afork-kicad-parts:DFN-8_L3.2-W3.1-P0.65-LS3.4-BL
- R2: footprint (none) -> Resistor_SMD:R_1206_3216Metric
- R30, R32, R4, R6: footprint (none) -> Resistor_SMD:R_0603_1608Metric
- U2: footprint :SOT-23-6_L2.9-W1.6-P0.95-LS2.8-TL -> esp32-bldc-foc:SOT-23-6_L2.9-W1.6-P0.95-LS2.8-TL
Changed lines of the file:
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@@
 			)
 		)
-		(property "Footprint" ""
+		(property "Footprint" "Resistor_SMD:R_0603_1608Metric"
 			(at 146.558 87.63 90)
 			(effects
@@
 			)
 		)
-		(property "Footprint" ":DFN-8_L3.2-W3.1-P0.65-LS3.4-BL"
+		(property "Footprint" "afork-kicad-parts:DFN-8_L3.2-W3.1-P0.65-LS3.4-BL"
 			(at 96.52 85.09 0)
 			(effects
@@
 			)
 		)
-		(property "Footprint" ""
+		(property "Footprint" "Capacitor_SMD:C_0603_1608Metric"
 			(at 69.85 86.36 0)
 			(effects
@@
 			)
 		)
-		(property "Footprint" ""
+		(property "Footprint" "Resistor_SMD:R_0603_1608Metric"
 			(at 78.74 81.788 90)
 			(effects
@@
 			)
 		)
-		(property "Footprint" ""
+		(property "Footprint" "Resistor_SMD:R_1206_3216Metric"
 			(at 116.84 94.488 90)
 			(effects
@@
 			)
 		)
-		(property "Footprint" ""
+		(property "Footprint" "Diode_SMD:D_SOD-323"
 			(at 69.85 66.04 0)
 			(effects
@@
 			)
 		)
-		(property "Footprint" ":DFN-8_L3.2-W3.1-P0.65-LS3.4-BL"
+		(property "Footprint" "afork-kicad-parts:DFN-8_L3.2-W3.1-P0.65-LS3.4-BL"
 			(at 96.52 59.69 0)
 			(effects
@@
 			)
 		)
-		(property "Footprint" ""
+		(property "Footprint" "Resistor_SMD:R_0603_1608Metric"
 			(at 78.74 107.188 90)
 			(effects
@@
 			)
 		)
-		(property "Footprint" ""
+		(property "Footprint" "Capacitor_SMD:C_0603_1608Metric"
 			(at 139.7 63.5 0)
 			(effects
@@
 			)
 		)
-		(property "Footprint" ":SOT-23-6_L2.9-W1.6-P0.95-LS2.8-TL"
+		(property "Footprint" "esp32-bldc-foc:SOT-23-6_L2.9-W1.6-P0.95-LS2.8-TL"
 			(at 132.08 85.09 0)
 			(effects
@@
 			)
 		)
-		(property "Footprint" ""
+		(property "Footprint" "Resistor_SMD:R_0603_1608Metric"
 			(at 143.002 100.33 90)
 			(effects

Commit message: Third cut of PCB.  Ready for BoM and routing
Parts:
- C25: footprint (none) -> Capacitor_SMD:C_1206_3216Metric
- Q16, Q18: footprint afork-kicad-parts:DFN-8_L3.2-W3.1-P0.65-LS3.4-BL -> esp32-bldc-foc:DFN-8_L3.2-W3.1-P0.65-LS3.4-BL
- U2: footprint esp32-bldc-foc:SOT-23-6_L2.9-W1.6-P0.95-LS2.8-TL -> Package_TO_SOT_SMD:SOT-23-6
Changed lines of the file:
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@@
 			)
 		)
-		(property "Footprint" "afork-kicad-parts:DFN-8_L3.2-W3.1-P0.65-LS3.4-BL"
+		(property "Footprint" "esp32-bldc-foc:DFN-8_L3.2-W3.1-P0.65-LS3.4-BL"
 			(at 96.52 85.09 0)
 			(effects
@@
 			)
 		)
-		(property "Footprint" ""
+		(property "Footprint" "Capacitor_SMD:C_1206_3216Metric"
 			(at 99.06 77.47 0)
 			(effects
@@
 			)
 		)
-		(property "Footprint" "afork-kicad-parts:DFN-8_L3.2-W3.1-P0.65-LS3.4-BL"
+		(property "Footprint" "esp32-bldc-foc:DFN-8_L3.2-W3.1-P0.65-LS3.4-BL"
 			(at 96.52 59.69 0)
 			(effects
@@
 			)
 		)
-		(property "Footprint" "esp32-bldc-foc:SOT-23-6_L2.9-W1.6-P0.95-LS2.8-TL"
+		(property "Footprint" "Package_TO_SOT_SMD:SOT-23-6"
 			(at 132.08 85.09 0)
 			(effects

Commit message: Remove "LCSC Part" field (I use just "LCSC")
Parts:
- Q16, Q18: LCSC (none) -> C2828592; LCSC Part C2828592 -> (none)
- U2: LCSC (none) -> C2058943; LCSC Part C2058943 -> (none)
Changed lines of the file:
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@@
 			)
 		)
-		(property "LCSC Part" "C2828592"
-			(at 96.52 87.63 0)
+		(property "LCSC" "C2828592"
+			(at 92.71 105.41 0)
 			(effects
 				(font
@@
 			)
 		)
-		(property "LCSC Part" "C2828592"
-			(at 96.52 62.23 0)
+		(property "LCSC" "C2828592"
+			(at 92.71 80.01 0)
 			(effects
 				(font
@@
 			)
 		)
-		(property "LCSC Part" "C2058943"
-			(at 132.08 87.63 0)
-			(effects
-				(font
+		(property "LCSC" "C2058943"
+			(at 132.08 74.93 0)
+			(effects
+				(font
